Commit message: added puma01_hardware_interface, and some other changes

File: puma01_description/urdf/puma01_sim.urdf (robot description, URDF)
Before this commit: robot puma01, 9 links, 8 joints
Joints:
- joint joint_4: limit lower=-1.92 upper=2.97 effort=10.0 velocity=5.0 -> lower=-1.92 upper=2.97 effort=50.0 velocity=5.0
- joint joint_5: limit lower=-1.74 upper=1.74 effort=10.0 velocity=5.0 -> lower=-1.74 upper=1.74 effort=50.0 velocity=5.0
- joint joint_6: limit lower=-4.64 upper=4.64 effort=10.0 velocity=5.0 -> lower=-4.64 upper=4.64 effort=50.0 velocity=5.0

Commit message: + vel and eff limits to sim controller & tweaked urdfs

File: puma01_description/urdf/puma01_sim.urdf (robot description, URDF)
Before this commit: robot puma01, 9 links, 8 joints
Joints:
- joint joint_1: limit lower=-2.79 upper=2.79 effort=80.0 velocity=5.0 -> lower=-2.79 upper=2.79 effort=150.0 velocity=10.0
- joint joint_2: limit lower=-3.93 upper=0.78 effort=80.0 velocity=5.0 -> lower=-3.93 upper=0.78 effort=150.0 velocity=10.0
- joint joint_3: limit lower=-0.78 upper=3.93 effort=80.0 velocity=5.0 -> lower=-0.78 upper=3.93 effort=150.0 velocity=10.0
- joint joint_4: limit lower=-1.92 upper=2.97 effort=50.0 velocity=5.0 -> lower=-1.92 upper=2.97 effort=150.0 velocity=10.0
- joint joint_5: limit lower=-1.74 upper=1.74 effort=50.0 velocity=5.0 -> lower=-1.74 upper=1.74 effort=150.0 velocity=10.0
- joint joint_6: limit lower=-4.64 upper=4.64 effort=50.0 velocity=5.0 -> lower=-4.64 upper=4.64 effort=150.0 velocity=10.0
