Commit message: IMPORTANT: fixed transformations in urdf

File: puma01_description/urdf/puma01.urdf (robot description, URDF)
Before this commit: robot puma01, 9 links, 8 joints
Joints:
- joint joint_1: origin xyz=0.0  0.62357 0.0  rpy=-1.57079632679 -1.57079632679 0.0 -> xyz=0.0  0.0 0.62357 rpy=0.0 0.0 0.0
- joint link_link0: origin xyz=0.0 0.0 0.0 rpy=1.57079632679 0.0 3.14 -> xyz=0.0 0.0 0.0 rpy=0.0 0.0 0.0

File: puma01_description/urdf/puma01_sim.urdf (robot description, URDF)
Before this commit: robot puma01, 9 links, 8 joints
Joints:
- joint joint_1: origin xyz=0.0  0.62357 0.0  rpy=-1.57079632679 -1.57079632679 0.0 -> xyz=0.0  0.0 0.62357 rpy=0.0 0.0 0.0
- joint link_link0: origin xyz=0.0 0.0 0.0 rpy=1.57079632679 0.0 3.14 -> xyz=0.0 0.0 0.0 rpy=0.0 0.0 0.0

Commit message: - tweaked usbcan wrapMsgData and getDataFromMsg; - added puma_parameters.h; - tweaked three_dof_test node; - added fake end-effector to module, but joystick failed to work properly;

File: puma01_description/urdf/puma01.urdf (robot description, URDF)
Before this commit: robot puma01, 9 links, 8 joints
Joints:
- joint joint_6_T: limit (none) -> lower=-0.01 upper=0.01 effort=1000.0 velocity=0.001; type fixed -> revolute

Commit message: - changed D-H parameters and urdf; - changed joint limits; - changed computed_torque_controller;

File: puma01_description/urdf/puma01.urdf (robot description, URDF)
Before this commit: robot puma01, 9 links, 8 joints
Joints:
- joint joint_2: limit lower=-3.93 upper=0.78 effort=150.0 velocity=10.0 -> lower=-2.32 upper=2.32 effort=150.0 velocity=10.0; origin xyz=0.0 0.2182 0.0 rpy=-1.57079632679 0.0 0.0 -> xyz=0.0 0.2182 0.0 rpy=-1.57079632679 -1.57079632679 0.0
- joint joint_3: limit lower=-0.78 upper=3.93 effort=150.0 velocity=10.0 -> lower=-2.478 upper=2.478 effort=150.0 velocity=10.0; origin xyz=0.4318 0.0 -0.0889 rpy=0.0 0.0 0.0 -> xyz=0.4318 0.0 -0.0889 rpy=0.0 0.0 1.57079632679

File: puma01_description/urdf/puma01_sim.urdf (robot description, URDF)
Before this commit: robot puma01, 9 links, 8 joints
Joints:
- joint joint_2: limit lower=-3.93 upper=0.78 effort=150.0 velocity=10.0 -> lower=-2.32 upper=2.32 effort=150.0 velocity=10.0; origin xyz=0.0 0.2182 0.0 rpy=-1.57079632679 0.0 0.0 -> xyz=0.0 0.2182 0.0 rpy=-1.57079632679 -1.57079632679 0.0
- joint joint_3: limit lower=-0.78 upper=3.93 effort=150.0 velocity=10.0 -> lower=-2.478 upper=2.478 effort=150.0 velocity=10.0; origin xyz=0.4318 0.0 -0.0889 rpy=0.0 0.0 0.0 -> xyz=0.4318 0.0 -0.0889 rpy=0.0 0.0 1.57079632679

Commit message: - added new moveit cfg package - tweaked computed torque - tweaked urdfs

File: puma01_description/urdf/puma01.urdf (robot description, URDF)
Before this commit: robot puma01, 9 links, 8 joints
Links:
- link link_T: mass 0.001 -> 0.0001
Joints:
- joint joint_6_T: limit lower=-0.01 upper=0.01 effort=1000.0 velocity=0.001 -> lower=0 upper=0 effort=1.0 velocity=1.0

Commit message: - added hwi_test node - solved "Missing joint_6_T state" warning

File: puma01_description/urdf/puma01.urdf (robot description, URDF)
Before this commit: robot puma01, 9 links, 8 joints
Joints:
- joint joint_6_T: limit lower=0 upper=0 effort=1.0 velocity=1.0 -> (none); type revolute -> fixed
